File: sfan.kicad_pcb (KiCad board)
At the start: 2 copper layers, 23 parts, among them J1 Conn_01x02_Male, J2 UART, J3 SWIM, J4 Barrel_Jack, Q1 Q_NPN_EBC, Q2 SI2300, U1 STM8S003F3U, U2 AMS1117-5.0

Commit message: pcb layout
Parts:
- removed RV1: 10K, Connector_PinHeader_1.27mm:PinHeader_1x03_P1.27mm_Vertical
- added C6: 104, Capacitor_SMD:C_0603_1608Metric, F.Cu at (127.8, 111.5)
- added C7: 104, Capacitor_SMD:C_0603_1608Metric, F.Cu at (107.7, 104.1)
- added C8: 104, Capacitor_SMD:C_0603_1608Metric, F.Cu at (107.7, 107.5)
- added C9: 22u, Capacitor_Tantalum_SMD:CP_EIA-3216-10_Kemet-I, F.Cu at (135.9, 105.9)
- added R6: 103, Resistor_SMD:R_0603_1608Metric, F.Cu at (130.0, 112.3)
- added R7: 103, Resistor_SMD:R_0603_1608Metric, F.Cu at (107.7, 101.1)
- added R8: 103, Resistor_SMD:R_0603_1608Metric, F.Cu at (107.7, 110.5)
- added R9: 103, Resistor_SMD:R_0603_1608Metric, F.Cu at (66.3, 105.4)
- added REF**: MountingHole_3.2mm_M3, MountingHole:MountingHole_3.2mm_M3, F.Cu at (156.0, 109.2)
- added REF**: MountingHole_3.2mm_M3, MountingHole:MountingHole_3.2mm_M3, F.Cu at (61.0, 109.2)
- added SW1: Rotary_Encoder_Switch, Rotary_Encoder:RotaryEncoder_Alps_EC11E-Switch_Vertical_H20mm, F.Cu at (111.0, 103.4)
- added TP1: TestPoint, TestPoint:TestPoint_Pad_D1.5mm, F.Cu at (63.8, 102.4)
- added TP2: TestPoint, TestPoint:TestPoint_Pad_D1.5mm, F.Cu at (72.9, 102.4)
- added TP3: TestPoint, TestPoint:TestPoint_Pad_D1.5mm, F.Cu at (66.3, 102.4)
- added TP4: TestPoint, TestPoint:TestPoint_Pad_D1.5mm, F.Cu at (61.2, 102.4)
- added TP5: TestPoint, TestPoint:TestPoint_Pad_D1.5mm, F.Cu at (78.0, 102.4)
- added TP6: TestPoint, TestPoint:TestPoint_Pad_D1.5mm, F.Cu at (75.4, 102.4)
- added TP7: TestPoint, TestPoint:TestPoint_Pad_D1.5mm, F.Cu at (80.5, 102.4)
- added TP8: TestPoint, TestPoint:TestPoint_Pad_D1.5mm, F.Cu at (68.8, 102.4)
- C3, C4: footprint efan:C_Radial_D5.0mm_H7.0mm_P2.00mm -> EFan:C_Radial_D5.0mm_H7.0mm_P2.00mm
- D1: footprint Diode_SMD:D_0603_1608Metric -> Diode_SMD:D_SMA
- D2, D3: footprint LED_SMD:LED_0603_1608Metric -> LED_SMD:LED_0805_2012Metric
- J1: footprint Connector_PinHeader_1.27mm:PinHeader_1x02_P1.27mm_Vertical -> Connector_PinHeader_2.54mm:PinHeader_1x02_P2.54mm_Vertical
- J2, J3: footprint Connector_PinHeader_1.27mm:PinHeader_1x04_P1.27mm_Vertical -> Connector_PinHeader_2.54mm:PinHeader_1x04_P2.54mm_Vertical
- J4: value Barrel_Jack -> Conn_01x02_Male; footprint Connector_BarrelJack:BarrelJack_CUI_PJ-063AH_Horizontal -> Connector_PinHeader_2.54mm:PinHeader_1x02_P2.54mm_Vertical
- moved C2 72.3 mm to (67.1, 109.0), turned to 180 degrees
- moved J4 62.9 mm to (149.1, 105.4), turned to 180 degrees
- moved R4 60.9 mm to (76.2, 105.4)
- moved J2 58.5 mm to (61.2, 99.1), turned to 90 degrees
- moved C3 53.5 mm to (148.8, 109.5), turned to 270 degrees
- moved R3 51.0 mm to (66.0, 112.3)
- moved U1 50.3 mm to (72.1, 107.7)
- moved U2 49.8 mm to (141.5, 108.2), turned to 90 degrees
- moved C5 49.8 mm to (69.3, 109.0), turned to 90 degrees
- moved Q2 47.8 mm to (80.3, 105.4), turned to 90 degrees
- moved D2 46.6 mm to (69.3, 112.3)
- moved J1 46.4 mm to (90.2, 99.3)
- moved R1 44.9 mm to (93.2, 112.3), turned to 270 degrees
- moved Q1 44.0 mm to (89.4, 107.2), turned to 270 degrees
- moved BZ1 41.7 mm to (99.3, 104.1), turned to 270 degrees
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Connections:
- net Net-(R2-Pad1) renamed /BEEP
- net Net-(R4-Pad1) renamed /PWM
- J4 pad 1: GND -> /+12V
- J4 pad 2: /+12V -> GND
- U1 pad 10: Net-(U1-Pad10) -> /PSBTN
- U1 pad 11: Net-(U1-Pad11) -> /REB
- U1 pad 12: Net-(U1-Pad12) -> /REA
Routing:
- net +5V: track 0.00 -> 98.3 mm, vias 0 -> 7
- net /+12V: track 0.00 -> 78.8 mm
- net /PSBTN: track 0.00 -> 63.9 mm
- net /REB: track 0.00 -> 41.1 mm
- net /REA: track 0.00 -> 41.1 mm
- net GND: track 0.00 -> 32.0 mm, vias 0 -> 10
- net /BEEP: track 0.00 -> 17.0 mm, vias 0 -> 2
- net Net-(C1-Pad2): track 0.00 -> 14.6 mm
- net Net-(J3-Pad4): track 0.00 -> 14.6 mm, vias 0 -> 2
- net Net-(D2-Pad1): track 0.00 -> 12.8 mm
- net Net-(BZ1-Pad2): track 0.00 -> 12.3 mm
- net Net-(J2-Pad2): track 0.00 -> 12.3 mm
- net Net-(J2-Pad3): track 0.00 -> 10.7 mm
- net Net-(J3-Pad3): track 0.00 -> 8.39 mm
- net Net-(Q1-Pad2): track 0.00 -> 4.29 mm
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- added copper zone on B.Cu, net +5V
- added copper zone on F.Cu, net +5V
- added copper zone on B.Cu, net GND
- added copper zone on F.Cu, net GND
Other:
- board outline added: 104.6 x 25.9 mm

Commit message: update refine
Parts:
- added REF**: Symbol_CC-Noncommercial_CopperTop_Small, Symbol:Symbol_CC-Noncommercial_CopperTop_Small, B.Cu at (151.2, 98.9)
- added REF**: Symbol_CC-Attribution_CopperTop_Small, Symbol:Symbol_CC-Attribution_CopperTop_Small, B.Cu at (157.2, 98.9)
- added REF**: KiCad-Logo2_5mm_SilkScreen, Symbol:KiCad-Logo2_5mm_SilkScreen, F.Cu at (139.8, 98.8)
- J1: value Conn_01x02_Male -> FAN
- J4: value Conn_01x02_Male -> 12V
- TP1: value TestPoint -> RX
- TP2: value TestPoint -> NRST
- TP3: value TestPoint -> TX
- TP4, TP5: value TestPoint -> GND
- TP6: value TestPoint -> SWIM
- TP7, TP8: value TestPoint -> 5V
- moved J4 3.07 mm to (148.7, 102.4), turned to 0 degrees
- renumbered J3 to SWD, J2 to UART
Routing:
- net /+12V: track 78.8 -> 80.2 mm
Other:
- board size 104.6 x 25.9 mm -> 104.6 x 18.7 mm
- board text added: "+"
- board text added: "-"
- board text added: "STM8S003F3U6"

Commit message: comply to jlc's 10cm limit
Parts:
- moved REF** 1.52 mm to (149.7, 98.9)
- moved REF** 1.52 mm to (155.7, 98.9)
Other:
- board size 104.6 x 18.7 mm -> 100 x 18.7 mm
Changed lines of the file:
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@@
-(kicad_pcb (version 20171130) (host pcbnew "(5.1.2-1)-1")
+(kicad_pcb (version 20171130) (host pcbnew "(5.1.2)-2")
   (general
     (thickness 1.6)
-    (drawings 10)
+    (drawings 11)
     (tracks 200)
     (zones 0)
@@
   )
   (setup
-    (last_trace_width 1)
+    (last_trace_width 0.25)
     (user_trace_width 0.5)
     (user_trace_width 1)
@@
       (usegerberadvancedattributes false)
       (creategerberjobfile false)
+      (gerberprecision 5)
       (excludeedgelayer true)
       (linewidth 0.100000)
@@
       (outputformat 1)
       (mirror false)
-      (drillshape 1)
+      (drillshape 0)
       (scaleselection 1)
-      (outputdirectory ""))
+      (outputdirectory "../gerber/sfan/"))
   )
   (net 0 "")
@@
   )
   (module Symbol:Symbol_CC-Noncommercial_CopperTop_Small (layer B.Cu)
-    (at 151.226 98.933)
+    (at 149.702 98.933)
     (descr "Symbol, CC-Noncommercial Alike, Copper Top, Small,")
     (tags "Symbol, CC-Noncommercial Alike, Copper Top, Small,")
@@
   )
   (module Symbol:Symbol_CC-Attribution_CopperTop_Small (layer B.Cu)
-    (at 157.226 98.933)
+    (at 155.702 98.933)
     (descr "Symbol, CC-Share Alike, Copper Top, Small,")
     (tags "Symbol, CC-Share Alike, Copper Top, Small,")
@@
     )
   )
+  (dimension 99.985603 (width 0.15) (layer Dwgs.User)
+    (gr_text "99.986 mm" (at 108.555833 118.101531 0.01455522364) (layer Dwgs.User)
+      (effects (font (size 1 1) (thickness 0.15)))
+    )
+    (feature1 (pts (xy 158.5476 114.0206) (xy 158.548452 117.375252)))
+    (feature2 (pts (xy 58.562 114.046) (xy 58.562852 117.400652)))
+    (crossbar (pts (xy 58.562703 116.814231) (xy 158.548303 116.788831)))
+    (arrow1a (pts (xy 158.548303 116.788831) (xy 157.421948 117.375538)))
+    (arrow1b (pts (xy 158.548303 116.788831) (xy 157.42165 116.202696)))
+    (arrow2a (pts (xy 58.562703 116.814231) (xy 59.689356 117.400366)))
+    (arrow2b (pts (xy 58.562703 116.814231) (xy 59.689058 116.227524)))
+  )
   (gr_text - (at 92.837 102.362) (layer F.SilkS)
     (effects (font (size 1 1) (thickness 0.25)))
@@
     (effects (font (size 1.5 1.5) (thickness 0.3)))
   )
-  (gr_line (start 56.134 114.046) (end 56.134 95.377) (layer Edge.Cuts) (width 0.05))
-  (gr_line (start 160.782 95.377) (end 160.782 114.046) (layer Edge.Cuts) (width 0.05))
-  (gr_line (start 56.134 95.377) (end 160.782 95.377) (layer Edge.Cuts) (width 0.05))
-  (gr_line (start 60.96 114.046) (end 56.134 114.046) (layer Edge.Cuts) (width 0.05))
-  (gr_line (start 60.96 114.046) (end 160.782 114.046) (layer Edge.Cuts) (width 0.05))
+  (gr_line (start 58.562 114.046) (end 58.562 95.377) (layer Edge.Cuts) (width 0.05))
+  (gr_line (start 158.5476 95.377) (end 158.5476 114.0206) (layer Edge.Cuts) (width 0.05))
+  (gr_line (start 58.562 95.377) (end 158.5476 95.377) (layer Edge.Cuts) (width 0.05))
+  (gr_line (start 60.96 114.046) (end 58.562 114.046) (layer Edge.Cuts) (width 0.05))
+  (gr_line (start 60.96 114.046) (end 158.5476 114.0206) (layer Edge.Cuts) (width 0.05))
   (via (at 96.774 107.696) (size 0.8) (drill 0.4) (layers F.Cu B.Cu) (net 0))
   (via (at 96.774 108.712) (size 0.8) (drill 0.4) (layers F.Cu B.Cu) (net 0))

Commit message: solder mask adj. this problem cost me 5 yuan and another round of production
Other:
- rule solder_mask_min_width: 0.25 -> 0.051
Changed lines of the file:
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@@
     (pad_drill 0.762)
     (pad_to_mask_clearance 0.051)
-    (solder_mask_min_width 0.25)
+    (solder_mask_min_width 0.051)
     (aux_axis_origin 0 0)
     (visible_elements 7FFFFFFF)
